Commit message: feat: ByteTrack 视觉检测集成 + 相机/机器人配置与 DWA 视觉接口
- 新增 bytetrack_ros: YOLOX+ByteTrack 桥接节点、检测图像 GUI
- 前视相机接入 Gazebo，f_oc 位姿与 DWA 订阅 /vision_dynamic_obstacles
- 机器人描述/相机/IMU 配置修正，DWA 与规划器参数调整
- 添加 README_UNCERTAINTY_FUSION_PLAN 阶段规划

Made-with: Cursor

File: robots/b2_description/urdf/b2_description.urdf (robot description, URDF)
Before this commit: robot b2_description, 26 links, 25 joints
Joints:
- joint f_oc_joint: origin xyz=0.39079 0 -0.013433 rpy=-1.5708 0 -1.5708 -> xyz=0.34918 0 0.17851 rpy=0 0 0

File: robots/b2_description/xacro/gazebo.xacro (robot description, xacro)
@@ -6,7 +6,7 @@
     <gazebo reference="imu_link">
       <sensor name="imu_sensor" type="imu">
-      <plugin filename="libgazebo_ros_imu_sensor.so" name="imu_plugin">
+      <plugin filename="libgazebo_ros_imu_sensor.so" name="b2_imu_plugin">
           <ros>
-            <namespace>/</namespace>
+            <namespace>/b2</namespace>
             <remapping>~/out:=imu</remapping>
           </ros>
@@ -72,34 +72,4 @@
       </sensor>
     </gazebo>
-    <ros2_control name="GazeboSystem" type="system">
-        <hardware>
-            <plugin>gazebo_ros2_control/GazeboSystem</plugin>
-        </hardware>
-        <xacro:macro name="joint_interface" params="joint_name torque_limit">
-            <joint name="${joint_name}">
-            <command_interface name="effort">
-                <param name="min">-${torque_limit}</param>
-                <param name="max">${torque_limit}</param>
-            </command_interface>
-            <state_interface name="position"/>
-            <state_interface name="velocity"/>
-            <state_interface name="effort"/>
-            </joint>
-        </xacro:macro>
-        <xacro:macro name="leg_joints" params="prefix">
-            <xacro:joint_interface joint_name="${prefix}_hip_joint" torque_limit="${hip_torque_max}"/>
-            <xacro:joint_interface joint_name="${prefix}_thigh_joint" torque_limit="${thigh_torque_max}"/>
-            <xacro:joint_interface joint_name="${prefix}_calf_joint" torque_limit="${calf_torque_max}"/>
-        </xacro:macro>
-        <xacro:leg_joints prefix="FR"/>
-        <xacro:leg_joints prefix="FL"/>
-        <xacro:leg_joints prefix="RR"/>
-        <xacro:leg_joints prefix="RL"/>
-    </ros2_control>
-    <gazebo>
-        <plugin name="gazebo_ros2_control" filename="libgazebo_ros2_control.so">
-            <parameters>$(find b2_description)/config/robot_control_ros2.yaml</parameters>
-        </plugin>
-    </gazebo>
     <gazebo reference="base_link">
         <!-- <material>Gazebo/Green</material> -->
@@ -216,3 +186,31 @@
         <kd  value="150.0"/>
     </gazebo>
+    <!-- Front camera mounted at official optical center link f_oc_link -->
+    <gazebo reference="f_oc_link">
+      <sensor name="front_camera" type="camera">
+        <update_rate>30</update_rate>
+        <camera>
+          <horizontal_fov>1.57</horizontal_fov>
+          <image>
+            <width>640</width>
+            <height>480</height>
+            <format>R8G8B8</format>
+          </image>
+          <clip>
+            <near>0.1</near>
+            <far>30.0</far>
+          </clip>
+        </camera>
+        <always_on>true</always_on>
+        <visualize>false</visualize>
+        <plugin name="front_camera_plugin" filename="libgazebo_ros_camera.so">
+          <ros>
+            <namespace>/</namespace>
+            <remapping>image_raw:=/front_camera/image_raw</remapping>
+            <remapping>camera_info:=/front_camera/camera_info</remapping>
+          </ros>
+          <frame_name>f_oc_link</frame_name>
+        </plugin>
+      </sensor>
+    </gazebo>
 </robot>

File: robots/b2_description/xacro/robot.xacro (robot description, xacro)
@@ -2,5 +2,5 @@
 <robot name="b2_description" xmlns:xacro="http://www.ros.org/wiki/xacro">
     <xacro:include filename="$(find b2_description)/xacro/gazebo_tf.xacro"/>
-    <!-- <xacro:include filename="$(find b2_description)/xacro/gazebo.xacro"/> -->
+    <xacro:include filename="$(find b2_description)/xacro/gazebo.xacro"/>
     <xacro:include filename="$(find b2_description)/urdf/b2_description.urdf"/>
     <xacro:include filename="$(find velodyne_description)/urdf/VLP-16.urdf.xacro" />
